File: ChargerShield.sch (EAGLE design)
At the start: 46 parts, among them IC1 LM324N, Q1 BD648, Q2 BC140-10, Q3 BC548, T2 BC548, X1 +5V, X2 Battery, X3 VCC

Commit message: update
Other:
- note added: "Battery Voltage"
- note added: "Buck"
- note added: "Charge- Current"
- note added: "Discharge- Current"
- note added: "User Interface"
- note added: "by Jedzia"
- note added: "work in progress;)"
- moved on the sheet: C4, Q2, R19

Commit message: reference voltage
Parts:
- removed Q3: BC548, transistor-npn:BC548
- added C5: 3µ3, rcl:CPOL-EUE5-5
- added IC2: TL431, AWJLEagleLib:TL431TO92
- added LED4: (no value), bigger:LED5MM_BIG
- added R21: 200, rcl:R-EU_0204/7
- added R22: 4k7, rcl:R-EU_0207/10
- added R23: 470, rcl:R-EU_0204/7
- added R24: 1k, rcl:R-EU_0207/10
- Q2: value BC140-10 -> BUZ11; device transistor-npn:BC140-10 -> transistor-fet:BUZ11
- R1, R3: value (none) -> 470
- R12: device rcl:R-EU_0207/10 -> rcl:R-EU_0207/12
- R13, R4: device rcl:R-EU_0207/12 -> rcl:R-EU_0207/10
- R19: value 200 -> 1k
- R20: value 1k -> 470; device rcl:R-EU_0204/7 -> rcl:R-EU_0207/10
- R9: device rcl:R-EU_0207/10 -> rcl:R-EU_0204/7
Connections:
- removed net DISC_1: Q3.E, R19.1
- removed net N$12: IC1B.+IN, Q2.C, R7.2
- new net N$25: Q2.S, R24.2, R7.1
- new net N$27: IC2.C, IC2.R, R21.1, R22.2
- new net N$28: R22.1, U$1.AREF
- new net N$29: C5.+, IC1B.+IN, R24.1
- net +5V: now also C4.1, IC1P.V+, R21.2; no longer LED2.A
- net GND: now also C5.-, IC2.A, LED2.C, LED4.C, R7.2; no longer Q2.E
- net N$13: now also Q2.D; no longer R7.1
- net N$18: now also Q2.G; no longer Q2.B
- net N$20: now also LED2.A; no longer Q3.B
- net N$21: now also LED4.A, R23.2; no longer LED2.C, Q3.C
- net PWM_DISCHARGE1: now also R19.1
- net PWM_DISCHARGE2: now also R23.1
- net VCC: no longer C4.1, IC1P.V+
Other:
- note removed: "what the fuck? muesste oben am R sein!"
- moved on the sheet: LED2, Q2, R19, R20, R7

Commit message: bigger power traces
Parts:
- added Q3: BUZ171, transistor-fet:BUZ171
- R5: device rcl:R-EU_0207/15 -> rcl:R-EU_0207/10
Connections:
- net N$7: now also Q3.G
- net N$9: now also Q3.S
- net VCC: now also Q3.D
Changed lines of the file:
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@@
 <part name="T2" library="transistor" deviceset="BC238" device="" value="BC548"/>
 <part name="R4" library="rcl" deviceset="R-EU_" device="0207/10" value="2k2"/>
-<part name="R5" library="rcl" deviceset="R-EU_" device="0207/15" value="1k"/>
+<part name="R5" library="rcl" deviceset="R-EU_" device="0207/10" value="1k"/>
 <part name="C3" library="rcl" deviceset="C-EU" device="025_050-025X075" value="15n/60V"/>
 <part name="GND4" library="supply1" deviceset="GND" device=""/>
@@
 <part name="R24" library="rcl" deviceset="R-EU_" device="0207/10" value="1k"/>
 <part name="C5" library="rcl" deviceset="CPOL-EU" device="E5-5" value="3µ3"/>
+<part name="Q3" library="transistor-fet" deviceset="BUZ171" device=""/>
 </parts>
 <sheets>
@@
 <instance part="R24" gate="G$1" x="64.77" y="57.15" rot="R180"/>
 <instance part="C5" gate="G$1" x="72.39" y="40.64"/>
+<instance part="Q3" gate="G$1" x="143.51" y="133.35"/>
 </instances>
 <busses>
@@
 <wire x1="109.22" y1="130.81" x2="109.22" y2="134.62" width="0.1524" layer="91"/>
 <pinref part="Q1" gate="G$1" pin="B"/>
-<wire x1="109.22" y1="130.81" x2="121.92" y2="130.81" width="0.1524" layer="91"/>
+<wire x1="109.22" y1="130.81" x2="118.11" y2="130.81" width="0.1524" layer="91"/>
 <junction x="109.22" y="130.81"/>
+<wire x1="118.11" y1="130.81" x2="121.92" y2="130.81" width="0.1524" layer="91"/>
+<wire x1="118.11" y1="130.81" x2="118.11" y2="123.19" width="0.1524" layer="91"/>
+<junction x="118.11" y="130.81"/>
+<wire x1="118.11" y1="123.19" x2="135.89" y2="123.19" width="0.1524" layer="91"/>
+<wire x1="135.89" y1="123.19" x2="135.89" y2="130.81" width="0.1524" layer="91"/>
+<pinref part="Q3" gate="G$1" pin="G"/>
+<wire x1="135.89" y1="130.81" x2="138.43" y2="130.81" width="0.1524" layer="91"/>
 </segment>
 </net>
@@
 <wire x1="129.54" y1="149.86" x2="129.54" y2="156.21" width="0.1524" layer="91"/>
 <pinref part="Q1" gate="G$1" pin="E"/>
-<wire x1="129.54" y1="138.43" x2="129.54" y2="149.86" width="0.1524" layer="91"/>
+<wire x1="129.54" y1="138.43" x2="129.54" y2="140.97" width="0.1524" layer="91"/>
 <junction x="129.54" y="149.86"/>
+<pinref part="Q3" gate="G$1" pin="D"/>
+<wire x1="129.54" y1="140.97" x2="129.54" y2="149.86" width="0.1524" layer="91"/>
+<wire x1="148.59" y1="135.89" x2="149.86" y2="135.89" width="0.1524" layer="91"/>
+<wire x1="149.86" y1="135.89" x2="149.86" y2="140.97" width="0.1524" layer="91"/>
+<wire x1="149.86" y1="140.97" x2="129.54" y2="140.97" width="0.1524" layer="91"/>
+<junction x="129.54" y="140.97"/>
 </segment>
 <segment>
@@
 <wire x1="129.54" y1="110.49" x2="129.54" y2="116.84" width="0.1524" layer="91"/>
 <pinref part="L1" gate="G$1" pin="1"/>
-<wire x1="129.54" y1="116.84" x2="129.54" y2="125.73" width="0.1524" layer="91"/>
+<wire x1="129.54" y1="116.84" x2="129.54" y2="120.65" width="0.1524" layer="91"/>
+<wire x1="129.54" y1="120.65" x2="129.54" y2="125.73" width="0.1524" layer="91"/>
 <wire x1="138.43" y1="116.84" x2="129.54" y2="116.84" width="0.1524" layer="91"/>
 <junction x="129.54" y="116.84"/>
-</segment>
-</net>
+<pinref part="Q3" gate="G$1" pin="S"/>
+<wire x1="148.59" y1="130.81" x2="149.86" y2="130.81" width="0.1524" layer="91"/>
+<wire x1="149.86" y1="130.81" x2="149.86" y2="120.65" width="0.1524" layer="91"/>
+<wire x1="149.86" y1="120.65" x2="129.54" y2="120.65" width="0.1524" layer="91"/>
+<junction x="129.54" y="120.65"/>
+</segment>
+</net>

Commit message: bigger board
Parts:
- added JP3: (no value), bigger:JP2E
- added R25: 4k7, rcl:R-EU_0204/7
- added U$2: DS1820TO92, Ava:DS1820TO92
- R19: device rcl:R-EU_0207/10 -> rcl:R-EU_0204/7
Connections:
- new net N$12: JP3.2, R25.1, U$1.D2, U$2.DQ
- net +5V: now also R25.2
- net GND: now also JP3.1, JP3.3, U$2.GND, U$2.VCC
- net PWM_CHARGE2: now also U$1.D11; no longer U$1.D9
- net PWM_DISCHARGE2: now also U$1.D9; no longer U$1.D11
Changed lines of the file:
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@@
 <part name="P+5" library="supply1" deviceset="VCC" device=""/>
 <part name="GND12" library="supply1" deviceset="GND" device=""/>
-<part name="R19" library="rcl" deviceset="R-EU_" device="0207/10" value="1k"/>
+<part name="R19" library="rcl" deviceset="R-EU_" device="0204/7" value="1k"/>
 <part name="R20" library="rcl" deviceset="R-EU_" device="0207/10" value="470"/>
 <part name="LED2" library="bigger" deviceset="LED" device="5MM_BIG"/>
@@
 <part name="C5" library="rcl" deviceset="CPOL-EU" device="E5-5" value="3µ3"/>
 <part name="Q3" library="transistor-fet" deviceset="BUZ171" device=""/>
+<part name="U$2" library="Ava" deviceset="DS1820" device="TO92"/>
+<part name="R25" library="rcl" deviceset="R-EU_" device="0204/7" value="4k7"/>
+<part name="P+8" library="supply1" deviceset="+5V" device=""/>
+<part name="GND14" library="supply1" deviceset="GND" device=""/>
+<part name="JP3" library="bigger" deviceset="JP2E" device=""/>
 </parts>
 <sheets>
@@
 <instance part="R23" gate="G$1" x="246.38" y="107.95" rot="MR270"/>
 <instance part="LED4" gate="G$1" x="246.38" y="97.79"/>
+<instance part="U$2" gate="G$1" x="195.58" y="59.69" rot="R270"/>
+<instance part="R25" gate="G$1" x="179.07" y="71.12" rot="R90"/>
+<instance part="P+8" gate="1" x="179.07" y="82.55"/>
+<instance part="GND14" gate="1" x="186.69" y="50.8"/>
+<instance part="JP3" gate="1" x="222.25" y="59.69" rot="R270"/>
 </instances>
 <busses>
@@
 <junction x="87.63" y="127"/>
 </segment>
+<segment>
+<pinref part="U$2" gate="G$1" pin="GND"/>
+<pinref part="GND14" gate="1" pin="GND"/>
+<wire x1="190.5" y1="62.23" x2="186.69" y2="62.23" width="0.1524" layer="91"/>
+<wire x1="186.69" y1="62.23" x2="186.69" y2="57.15" width="0.1524" layer="91"/>
+<pinref part="U$2" gate="G$1" pin="VCC"/>
+<wire x1="186.69" y1="57.15" x2="186.69" y2="53.34" width="0.1524" layer="91"/>
+<wire x1="190.5" y1="57.15" x2="189.23" y2="57.15" width="0.1524" layer="91"/>
+<junction x="186.69" y="57.15"/>
+<wire x1="189.23" y1="57.15" x2="186.69" y2="57.15" width="0.1524" layer="91"/>
+<wire x1="186.69" y1="62.23" x2="186.69" y2="68.58" width="0.1524" layer="91"/>
+<junction x="186.69" y="62.23"/>
+<wire x1="186.69" y1="68.58" x2="215.9" y2="68.58" width="0.1524" layer="91"/>
+<wire x1="215.9" y1="68.58" x2="215.9" y2="62.23" width="0.1524" layer="91"/>
+<pinref part="JP3" gate="1" pin="1"/>
+<wire x1="215.9" y1="62.23" x2="219.71" y2="62.23" width="0.1524" layer="91"/>
+<wire x1="189.23" y1="57.15" x2="189.23" y2="53.34" width="0.1524" layer="91"/>
+<junction x="189.23" y="57.15"/>
+<wire x1="189.23" y1="53.34" x2="214.63" y2="53.34" width="0.1524" layer="91"/>
+<wire x1="214.63" y1="53.34" x2="214.63" y2="57.15" width="0.1524" layer="91"/>
+<pinref part="JP3" gate="1" pin="3"/>
+<wire x1="214.63" y1="57.15" x2="219.71" y2="57.15" width="0.1524" layer="91"/>
+</segment>
 </net>
 <net name="N$1" class="0">
@@
 <wire x1="214.63" y1="171.45" x2="214.63" y2="172.72" width="0.1524" layer="91"/>
 <wire x1="214.63" y1="172.72" x2="238.76" y2="172.72" width="0.1524" layer="91"/>
+</segment>
+<segment>
+<pinref part="P+8" gate="1" pin="+5V"/>
+<pinref part="R25" gate="G$1" pin="2"/>
+<wire x1="179.07" y1="80.01" x2="179.07" y2="76.2" width="0.1524" layer="91"/>
 </segment>
 </net>
@@
 <wire x1="191.77" y1="129.54" x2="236.22" y2="129.54" width="0.1524" layer="91"/>
 <wire x1="236.22" y1="129.54" x2="236.22" y2="113.03" width="0.1524" layer="91"/>
-<label x="193.04" y="137.16" size="1.778" layer="95" xref="yes"/>
+<label x="228.6" y="129.54" size="1.778" layer="95" xref="yes"/>
 </segment>
 </net>
@@
 <net name="PWM_CHARGE2" class="0">
 <segment>
-<pinref part="U$1" gate="G$1" pin="D9"/>
-<wire x1="152.4" y1="134.62" x2="167.64" y2="134.62" width="0.1524" layer="91"/>
-<label x="167.64" y="134.62" size="1.778" layer="95" xref="yes"/>
+<label x="173.99" y="139.7" size="1.778" layer="95" xref="yes"/>
+<pinref part="U$1" gate="G$1" pin="D11"/>
+<wire x1="173.99" y1="139.7" x2="152.4" y2="139.7" width="0.1524" layer="91"/>
 </segment>
 </net>
@@
 <net name="PWM_DISCHARGE2" class="0">
 <segment>
-<pinref part="U$1" gate="G$1" pin="D11"/>
-<wire x1="152.4" y1="139.7" x2="167.64" y2="139.7" width="0.1524" layer="91"/>
-<label x="168.91" y="140.97" size="1.778" layer="95" xref="yes"/>
-<wire x1="167.64" y1="139.7" x2="167.64" y2="140.97" width="0.1524" layer="91"/>
+<label x="233.68" y="134.62" size="1.778" layer="95" xref="yes"/>
 <pinref part="R23" gate="G$1" pin="1"/>
-<wire x1="246.38" y1="140.97" x2="246.38" y2="113.03" width="0.1524" layer="91"/>
-<wire x1="167.64" y1="140.97" x2="246.38" y2="140.97" width="0.1524" layer="91"/>
+<wire x1="246.38" y1="134.62" x2="246.38" y2="113.03" width="0.1524" layer="91"/>
+<wire x1="152.4" y1="134.62" x2="246.38" y2="134.62" width="0.1524" layer="91"/>
+<pinref part="U$1" gate="G$1" pin="D9"/>
 </segment>
 </net>
@@
 </segment>
 </net>
+<net name="N$12" class="0">
+<segment>
+<pinref part="U$1" gate="G$1" pin="D2"/>
+<wire x1="152.4" y1="114.3" x2="173.99" y2="114.3" width="0.1524" layer="91"/>
+<wire x1="173.99" y1="114.3" x2="173.99" y2="59.69" width="0.1524" layer="91"/>
+<pinref part="U$2" gate="G$1" pin="DQ"/>
+<wire x1="173.99" y1="59.69" x2="179.07" y2="59.69" width="0.1524" layer="91"/>
+<pinref part="R25" gate="G$1" pin="1"/>
+<wire x1="179.07" y1="59.69" x2="189.23" y2="59.69" width="0.1524" layer="91"/>
+<wire x1="189.23" y1="59.69" x2="190.5" y2="59.69" width="0.1524" layer="91"/>
+<wire x1="179.07" y1="66.04" x2="179.07" y2="59.69" width="0.1524" layer="91"/>
+<junction x="179.07" y="59.69"/>
+<wire x1="189.23" y1="59.69" x2="189.23" y2="66.04" width="0.1524" layer="91"/>
+<junction x="189.23" y="59.69"/>
+<wire x1="189.23" y1="66.04" x2="214.63" y2="66.04" width="0.1524" layer="91"/>
+<wire x1="214.63" y1="66.04" x2="214.63" y2="59.69" width="0.1524" layer="91"/>
+<pinref part="JP3" gate="1" pin="2"/>
+<wire x1="214.63" y1="59.69" x2="219.71" y2="59.69" width="0.1524" layer="91"/>
+</segment>
+</net>
