File: ChargerShieldwFront.brd (EAGLE design)
At the start: 135.9 x 134.6 mm, 58 parts, among them IC1 LM324N, IC2 TL431, Q1 BD648, Q2 BUZ11, Q3 BUZ171, T2 BC548, X1 +5V, X2 Battery, X3 VCC

Commit message: update
Parts:
- R1: device rcl:0207/10 -> rcl:0207/12
- R19: device rcl:0204/7 -> rcl:0207/12
- moved S1 28.4 mm to (47.0, 97.8)
- moved S4 28.4 mm to (21.6, 97.8)
- moved IC2 18.5 mm to (12.7, 36.8), turned to 0 degrees
- moved S2 16.3 mm to (39.4, 97.8)
- moved S3 16.3 mm to (29.2, 97.8)
- moved LED2 12.7 mm to (44.5, 128.3)
- moved LED4 12.7 mm to (35.6, 128.3)
- moved LED1 12.7 mm to (44.5, 113.0)
- moved LED3 12.7 mm to (35.6, 113.0)
- moved R1 12.7 mm to (17.8, 105.4)
- moved R20 12.7 mm to (29.2, 120.7)
- moved R23 12.7 mm to (29.2, 123.2)
- moved R3 12.7 mm to (29.2, 118.1)
- moved U$3 12.7 mm to (40.6, 85.1)
- moved U$6 12.7 mm to (17.8, 85.1)
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Routing:
- net N$19: track 0.00 -> 115.0 mm
- net PWM_DISCHARGE2: track 0.25 -> 74.5 mm
- net PWM_DISCHARGE1: track 3.33 -> 63.8 mm
- net +5V: track 59.0 -> 87.2 mm
- net N$1: track 0.00 -> 24.3 mm
- net N$32: track 0.00 -> 23.5 mm
- net N$22: track 0.00 -> 16.6 mm
- net N$3: track 0.00 -> 10.9 mm
- net N$4: track 0.00 -> 10.1 mm
- net N$8: track 57.0 -> 64.6 mm
- net N$12: track 23.3 -> 30.9 mm
- net N$13: track 104.7 -> 112.3 mm
- net I_SENSE: track 55.0 -> 62.0 mm
- net N$36: track 53.1 -> 59.7 mm
- net GND: track 10.9 -> 15.4 mm
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Other:
- board size 135.9 x 134.6 mm -> 135.9 x 147.3 mm
