File: ChargerShieldwFront.sch (EAGLE design)
At the start: 60 parts, among them IC1 LM324N, IC2 TL431, Q1 BD648, Q2 BUZ11, Q3 BUZ171, T2 BC548, X1 +5V, X2 Battery, X3 VCC

Commit message: update
Parts:
- R1: device rcl:R-EU_0207/10 -> rcl:R-EU_0207/12
- R19: device rcl:R-EU_0204/7 -> rcl:R-EU_0207/12
Changed lines of the file:
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@@
 <setting verticaltext="up"/>
 </settings>
-<grid distance="0.05" unitdist="inch" unit="mm" style="lines" multiple="1" display="yes" altdistance="0.025" altunitdist="inch" altunit="mm"/>
+<grid distance="0.1" unitdist="inch" unit="inch" style="lines" multiple="1" display="no" altdistance="0.01" altunitdist="inch" altunit="inch"/>
 <layers>
 <layer number="1" name="Top" color="4" fill="1" visible="yes" active="no"/>
@@
 <part name="P+1" library="supply1" deviceset="+5V" device=""/>
 <part name="P+2" library="supply1" deviceset="+5V" device=""/>
-<part name="R1" library="rcl" deviceset="R-EU_" device="0207/10" value="470"/>
+<part name="R1" library="rcl" deviceset="R-EU_" device="0207/12" value="470"/>
 <part name="U$1" library="arduino-long" deviceset="ARDUINOR3" device="BPLACE-LONG" value="ARDUINOR3BPLACE-LONG"/>
 <part name="X1" library="con-wago-500" deviceset="W237-102" device="" value="+5V"/>
@@
 <part name="P+5" library="supply1" deviceset="VCC" device=""/>
 <part name="GND12" library="supply1" deviceset="GND" device=""/>
-<part name="R19" library="rcl" deviceset="R-EU_" device="0204/7" value="1k"/>
+<part name="R19" library="rcl" deviceset="R-EU_" device="0207/12" value="1k"/>
 <part name="R20" library="rcl" deviceset="R-EU_" device="0207/10" value="470"/>
 <part name="LED2" library="bigger" deviceset="LED" device="5MM_BIG"/>
