File: ChargerShieldwFront01.sch (EAGLE design)
At the start: 94 parts, among them IC1 TL431, IC2 LM324N, Q1 BUZ11BH, Q2 BD648, Q3 BUZ171, Q4 BUZ11BH, Q5 BD648, Q6 BUZ171, T1 BC548, T2 BC548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

Commit message: all I_batt differential
Parts:
- added R43: 100k, rcl:R-EU_0207/10
- R29: device rcl:R-EU_0207/10 -> rcl:R-EU_0204/7
- R38: device rcl:R-EU_0204/7 -> rcl:R-EU_0207/15
- R39: value 1k -> 10k
Connections:
- net I_SENSE2 renamed I2_SENSE+
- new net I2_SENSE-: R38.1, X4-5.KL
- net GND: now also R43.2; no longer R38.1
- net I_BATT2: now also C8.+
- net N$46: now also R43.1; no longer C8.+
Other:
- moved on the sheet: C8, R37, R38
Changed lines of the file:
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@@
 <part name="JP5" library="bigger" deviceset="JP1E" device=""/>
 <part name="R37" library="rcl" deviceset="R-EU_" device="0204/7" value="100k"/>
-<part name="R38" library="rcl" deviceset="R-EU_" device="0204/7" value="10k"/>
+<part name="R38" library="rcl" deviceset="R-EU_" device="0207/15" value="10k"/>
 <part name="GND19" library="supply1" deviceset="GND" device=""/>
 <part name="XR32" library="lt-spice-simulation" deviceset="RES_RLOAD" device="" value="0R1"/>
 <part name="R26" library="rcl" deviceset="R-EU_" device="0414/15" value="1R666"/>
 <part name="GND20" library="supply1" deviceset="GND" device=""/>
-<part name="R29" library="rcl" deviceset="R-EU_" device="0207/10" value="100k"/>
+<part name="R29" library="rcl" deviceset="R-EU_" device="0204/7" value="100k"/>
 <part name="R36" library="rcl" deviceset="R-EU_" device="0207/12" value="1k"/>
 <part name="R41" library="rcl" deviceset="R-EU_" device="0207/10" value="100k"/>
 <part name="C9" library="rcl" deviceset="CPOL-EU" device="E5-5" value="10µ"/>
-<part name="R39" library="rcl" deviceset="R-EU_" device="0207/10" value="1k"/>
+<part name="R39" library="rcl" deviceset="R-EU_" device="0207/10" value="10k"/>
 <part name="C8" library="rcl" deviceset="CPOL-EU" device="E5-5" value="3µ3"/>
 <part name="R31" library="rcl" deviceset="R-EU_" device="0207/10" value="100k"/>
@@
 <part name="FRAME3" library="frames" deviceset="DINA4_L" device=""/>
 <part name="R42" library="rcl" deviceset="R-EU_" device="0204/7" value="100k"/>
+<part name="R43" library="rcl" deviceset="R-EU_" device="0207/10" value="100k"/>
+<part name="GND18" library="supply1" deviceset="GND" device=""/>
 </parts>
 <sheets>
@@
 <instance part="L2" gate="G$1" x="139.7" y="130.81" rot="R90"/>
 <instance part="V2" gate="G$1" x="240.03" y="127"/>
-<instance part="GND15" gate="1" x="179.07" y="82.55"/>
+<instance part="GND15" gate="1" x="130.81" y="80.01"/>
 <instance part="D4" gate="1" x="176.53" y="138.43" rot="R270"/>
 <instance part="JP4" gate="A" x="187.96" y="139.7" rot="R270"/>
@@
 <instance part="GND17" gate="1" x="207.01" y="82.55"/>
 <instance part="JP5" gate="A" x="200.66" y="139.7" rot="R270"/>
-<instance part="R37" gate="G$1" x="147.32" y="83.82" rot="R90"/>
-<instance part="R38" gate="G$1" x="147.32" y="64.77" rot="R90"/>
+<instance part="R37" gate="G$1" x="161.29" y="81.28" rot="R180"/>
+<instance part="R38" gate="G$1" x="189.23" y="81.28" rot="R180"/>
 <instance part="GND19" gate="1" x="147.32" y="33.02"/>
 <instance part="XR32" gate="G$1" x="237.49" y="106.68"/>
@@
 <instance part="C9" gate="G$1" x="224.79" y="148.59"/>
 <instance part="R39" gate="G$1" x="187.96" y="97.79"/>
-<instance part="C8" gate="G$1" x="179.07" y="92.71"/>
+<instance part="C8" gate="G$1" x="130.81" y="90.17"/>
 <instance part="R31" gate="G$1" x="95.25" y="57.15" rot="R90"/>
 <instance part="R33" gate="G$1" x="99.06" y="44.45" rot="R90"/>
@@
 <instance part="X4" gate="-5" x="219.71" y="106.68" rot="R180"/>
 <instance part="X4" gate="-6" x="219.71" y="86.36" rot="R180"/>
+<instance part="R43" gate="G$1" x="179.07" y="88.9" rot="R270"/>
+<instance part="GND18" gate="1" x="179.07" y="74.93"/>
 </instances>
 <busses>
@@
 </segment>
 <segment>
-<pinref part="R38" gate="G$1" pin="1"/>
-<pinref part="GND19" gate="1" pin="GND"/>
-<wire x1="147.32" y1="59.69" x2="147.32" y2="35.56" width="0.1524" layer="91"/>
-</segment>
-<segment>
 <pinref part="C8" gate="G$1" pin="-"/>
 <pinref part="GND15" gate="1" pin="GND"/>
-<wire x1="179.07" y1="87.63" x2="179.07" y2="85.09" width="0.1524" layer="91"/>
+<wire x1="130.81" y1="85.09" x2="130.81" y2="82.55" width="0.1524" layer="91"/>
 </segment>
 <segment>
@@
 <wire x1="68.58" y1="36.83" x2="54.61" y2="36.83" width="0.1524" layer="91"/>
 <junction x="54.61" y="36.83"/>
+</segment>
+<segment>
+<pinref part="R43" gate="G$1" pin="2"/>
+<pinref part="GND18" gate="1" pin="GND"/>
+<wire x1="179.07" y1="83.82" x2="179.07" y2="77.47" width="0.1524" layer="91"/>
 </segment>
 </net>
@@
 <pinref part="R37" gate="G$1" pin="2"/>
 <wire x1="153.67" y1="95.25" x2="147.32" y2="95.25" width="0.1524" layer="91"/>
-<wire x1="147.32" y1="95.25" x2="147.32" y2="88.9" width="0.1524" layer="91"/>
+<wire x1="147.32" y1="95.25" x2="147.32" y2="81.28" width="0.1524" layer="91"/>
+<wire x1="147.32" y1="81.28" x2="156.21" y2="81.28" width="0.1524" layer="91"/>
 <wire x1="147.32" y1="95.25" x2="143.51" y2="95.25" width="0.1524" layer="91"/>
 <junction x="147.32" y="95.25"/>
@@
 <segment>
 <pinref part="R37" gate="G$1" pin="1"/>
-<wire x1="147.32" y1="78.74" x2="147.32" y2="74.93" width="0.1524" layer="91"/>
-<wire x1="147.32" y1="74.93" x2="173.99" y2="74.93" width="0.1524" layer="91"/>
-<wire x1="173.99" y1="74.93" x2="173.99" y2="92.71" width="0.1524" layer="91"/>
+<wire x1="166.37" y1="81.28" x2="173.99" y2="81.28" width="0.1524" layer="91"/>
+<wire x1="173.99" y1="81.28" x2="173.99" y2="92.71" width="0.1524" layer="91"/>
 <wire x1="173.99" y1="92.71" x2="168.91" y2="92.71" width="0.1524" layer="91"/>
 <pinref part="R38" gate="G$1" pin="2"/>
-<wire x1="147.32" y1="69.85" x2="147.32" y2="74.93" width="0.1524" layer="91"/>
-<junction x="147.32" y="74.93"/>
+<wire x1="184.15" y1="81.28" x2="173.99" y2="81.28" width="0.1524" layer="91"/>
+<junction x="173.99" y="81.28"/>
 <pinref part="IC2" gate="C" pin="-IN"/>
 </segment>
@@
 <wire x1="168.91" y1="97.79" x2="179.07" y2="97.79" width="0.1524" layer="91"/>
 <pinref part="R39" gate="G$1" pin="1"/>
-<pinref part="C8" gate="G$1" pin="+"/>
+<pinref part="IC2" gate="C" pin="+IN"/>
+<pinref part="R43" gate="G$1" pin="1"/>
 <wire x1="179.07" y1="97.79" x2="182.88" y2="97.79" width="0.1524" layer="91"/>
-<wire x1="179.07" y1="97.79" x2="179.07" y2="95.25" width="0.1524" layer="91"/>
+<wire x1="179.07" y1="97.79" x2="179.07" y2="93.98" width="0.1524" layer="91"/>
 <junction x="179.07" y="97.79"/>
-<pinref part="IC2" gate="C" pin="+IN"/>
 </segment>
 </net>
@@
 <segment>
 <pinref part="R36" gate="G$1" pin="1"/>
-<wire x1="133.35" y1="95.25" x2="129.54" y2="95.25" width="0.1524" layer="91"/>
+<wire x1="133.35" y1="95.25" x2="130.81" y2="95.25" width="0.1524" layer="91"/>
 <label x="129.54" y="95.25" size="2.54" layer="95" rot="R180" xref="yes"/>
-</segment>
-</net>
-<net name="I_SENSE2" class="0">
+<pinref part="C8" gate="G$1" pin="+"/>
+<wire x1="130.81" y1="95.25" x2="129.54" y2="95.25" width="0.1524" layer="91"/>
+<wire x1="130.81" y1="95.25" x2="130.81" y2="92.71" width="0.1524" layer="91"/>
+<junction x="130.81" y="95.25"/>
+</segment>
+</net>
+<net name="I2_SENSE+" class="0">
 <segment>
 <pinref part="V2" gate="G$1" pin="-"/>
@@
 </segment>
 </net>
+<net name="I2_SENSE-" class="0">
+<segment>
+<pinref part="R38" gate="G$1" pin="1"/>
+<wire x1="194.31" y1="81.28" x2="198.12" y2="81.28" width="0.1524" layer="91"/>
+<wire x1="198.12" y1="81.28" x2="198.12" y2="106.68" width="0.1524" layer="91"/>
+<pinref part="X4" gate="-5" pin="KL"/>
+<wire x1="198.12" y1="106.68" x2="214.63" y2="106.68" width="0.1524" layer="91"/>
+<wire x1="214.63" y1="106.68" x2="229.87" y2="106.68" width="0.1524" layer="91"/>
+<wire x1="229.87" y1="106.68" x2="229.87" y2="88.9" width="0.1524" layer="91"/>
+<wire x1="229.87" y1="88.9" x2="237.49" y2="88.9" width="0.1524" layer="91"/>
+<junction x="214.63" y="106.68"/>
+<label x="243.84" y="88.9" size="1.778" layer="95" xref="yes"/>
+</segment>
+</net>

Commit message: arrangement
Parts:
- R12: device rcl:R-EU_0207/10 -> rcl:R-EU_0204/7
Changed lines of the file:
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@@
 <part name="R9" library="rcl" deviceset="R-EU_" device="0414/15" value="1R666"/>
 <part name="GND10" library="supply1" deviceset="GND" device=""/>
-<part name="R12" library="rcl" deviceset="R-EU_" device="0207/10" value="100k"/>
+<part name="R12" library="rcl" deviceset="R-EU_" device="0204/7" value="100k"/>
 <part name="R19" library="rcl" deviceset="R-EU_" device="0207/12" value="1k"/>
 <part name="R24" library="rcl" deviceset="R-EU_" device="0207/10" value="100k"/>
