File: ChargerShieldExpA.brd (EAGLE design)
At the start: 161.3 x 99.1 mm, 94 parts, among them IC1 LM324N, IC2 TL431, Q1 BD648, Q2 BUZ11, Q3 BUZ171, Q4 IRFZ48Z, T2 BC548, X1 +Vin, X2 Battery, X3 VCC

Commit message: tidy up
Parts:
- added JP20: (no value), bigger:JP2
- added JP21, JP22: (no value), bigger:JP1
- moved U$2 31.8 mm to (47.0, 37.5), turned to 180 degrees
- moved JP3 29.1 mm to (45.1, 42.5), turned to 180 degrees
- moved D1 9.67 mm to (104.1, 36.8), turned to 90 degrees
- moved C6 6.35 mm to (104.1, 45.7)
- moved JP17 5.08 mm to (8.89, -2.54)
- moved JP18 5.08 mm to (8.89, -7.62)
- moved R25 3.24 mm to (39.4, 38.7), turned to 90 degrees
- moved R4 2.54 mm to (71.1, 61.0)
- moved Q4 1.27 mm to (81.3, 38.1)
- moved R26 1.27 mm to (-6.99, 50.8)
- moved R27 1.27 mm to (-6.99, 48.3)
Connections:
- removed net GND2: LED1.K, LED2.K, LED3.K, LED4.K, LED5.K, LED6.K, S1.1, S2.1, S3.1, S4.1, S5.1, S6.1, U$3.1, U$6.1
- new net N$52: JP21.1, U$1.D0
- new net N$53: JP22.1, U$1.RESET
- net +5V: now also JP3.3, U$2.VDD
- net GND: now also JP22.2, LED1.K, LED2.K, LED3.K, LED4.K, LED5.K, LED6.K, S1.1, S2.1, S3.1, S4.1, S5.1, S6.1, U$3.1, U$6.1; no longer JP3.3, U$2.VDD
- net I_BATT2: now also JP20.2
- net I_DISC2: now also JP20.3
- net N$37: now also U$1.D6
- net N$38: now also U$1.SDA
- net N$41: now also R27.1, U$1.SCL, U$5.7, U$6.7; no longer R26.1, U$5.6, U$6.6
- net N$42: now also JP21.2, R26.1, U$1.D1, U$5.6, U$6.6; no longer R27.1, U$5.7, U$6.7
- net U_BATT2: now also JP20.1
Routing:
- net GND: track 134.7 -> 195.0 mm, vias 7 -> 8
- net N$42: track 68.3 -> 104.9 mm
- net N$12: track 67.9 -> 35.8 mm
- net N$38: track 139.8 -> 164.2 mm, vias 0 -> 2
- net PWM_CHARGE1: track 15.2 -> 35.6 mm
- net N$37: track 167.3 -> 186.3 mm, vias 0 -> 2
- net N$41: track 52.6 -> 68.2 mm, vias 2 -> 4
- net +5V: track 107.6 -> 121.1 mm
- net GND2: track 13.3 -> 0.00 mm, vias 1 -> 0
- net N$9: track 57.6 -> 44.9 mm
- net N$19: track 176.0 -> 183.9 mm
- net N$53: track 0.00 -> 7.62 mm
- net N$18: track 78.2 -> 84.9 mm
- net U_BATT2: track 0.00 -> 6.35 mm
- net I_DISC2: track 0.00 -> 6.35 mm
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- removed copper zone on layer 16, net GND2

Commit message: internal current sense shunt
Parts:
- added JP23, JP24: (no value), bigger:JP1
- added R39: 1R666, rcl:0414/15
- moved R5 11.4 mm to (94.0, 47.0)
- moved T2 11.4 mm to (87.6, 49.5)
- moved R11 8.89 mm to (96.5, 54.6)
- moved R4 6.84 mm to (73.7, 54.6)
- moved R6 5.08 mm to (104.1, 50.8)
Connections:
- new net N$54: JP24.1, JP6.2, X2.4
- net GND: now also JP23.2, R39.2
- net I1_SENSE+: now also JP24.2, R39.1, X2.3; no longer JP6.2, X2.4
- net I1_SENSE-: now also JP23.1
Routing:
- net N$54: track 0.00 -> 69.1 mm, vias 0 -> 2
- net I1_SENSE+: track 62.3 -> 17.8 mm, vias 2 -> 0
- net N$7: track 108.6 -> 94.7 mm
- net PWM_CHARGE1: track 35.6 -> 44.5 mm
- net N$13: track 130.8 -> 126.2 mm
- net N$5: track 16.1 -> 13.3 mm

Commit message: first layout
Parts:
- moved R5 3.81 mm to (94.0, 50.8)
- moved R6 2.54 mm to (104.1, 48.3)
- moved T2 1.80 mm to (86.4, 50.8), turned to 90 degrees
- moved R11 1.27 mm to (95.2, 54.6)
Routing:
- net N$7: track 94.7 -> 88.3 mm
- net N$6: track 5.08 -> 3.81 mm
- net N$26: track 147.3 -> 148.5 mm
- net N$5: track 13.3 -> 12.7 mm
Changed lines of the file:
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@@
 <setting verticaltext="up"/>
 </settings>
-<grid distance="2.54" unitdist="mm" unit="mm" style="lines" multiple="1" display="yes" altdistance="1.27" altunitdist="mm" altunit="mm"/>
+<grid distance="0.05" unitdist="inch" unit="mm" style="lines" multiple="1" display="yes" altdistance="0.025" altunitdist="inch" altunit="mm"/>
 <layers>
 <layer number="1" name="Top" color="4" fill="1" visible="yes" active="yes"/>
@@
 <element name="S1" library="bigger" package="TACTILE-PTH-UMSE" value="Down" x="-34.29" y="44.45" rot="R270"/>
 <element name="S2" library="bigger" package="TACTILE-PTH-UMSE" value="Up" x="-19.05" y="44.45" rot="R270"/>
-<element name="T2" library="transistor" package="TO92" value="BC548" x="87.63" y="49.53"/>
+<element name="T2" library="transistor" package="TO92" value="BC548" x="86.36" y="50.8" rot="R90"/>
 <element name="R4" library="rcl" package="0207/15" value="2k2" x="73.66" y="54.61"/>
-<element name="R5" library="rcl" package="0207/10" value="1k" x="93.98" y="46.99"/>
+<element name="R5" library="rcl" package="0207/10" value="1k" x="93.98" y="50.8"/>
 <element name="C3" library="rcl" package="C025_050-025X075" value="15n/60V" x="71.12" y="25.4" rot="R90"/>
-<element name="R6" library="rcl" package="0207/10" value="1k" x="104.14" y="50.8"/>
+<element name="R6" library="rcl" package="0207/10" value="1k" x="104.14" y="48.26"/>
 <element name="Q1" library="transistor-pnp" package="TO220" value="BD648" x="104.14" y="21.59" rot="R180"/>
 <element name="D1" library="diode" package="DO35-7" value="" x="104.14" y="36.83" rot="R90"/>
@@
 <element name="R9" library="rcl" package="0207/10" value="10k" x="64.77" y="30.48" rot="R270"/>
 <element name="R7" library="rcl" package="0414/15" value="1R666" x="53.34" y="-11.43" rot="R180"/>
-<element name="R11" library="rcl" package="0207/10" value="100k" x="96.52" y="54.61" rot="R180"/>
+<element name="R11" library="rcl" package="0207/10" value="100k" x="95.25" y="54.61" rot="R180"/>
 <element name="R12" library="rcl" package="0207/12" value="1k" x="46.99" y="11.43" rot="R180"/>
 <element name="R13" library="rcl" package="0207/10" value="100k" x="50.8" y="19.05" rot="R270"/>
@@
 <contactref element="T2" pad="2"/>
 <contactref element="R11" pad="2"/>
-<wire x1="91.44" y1="54.61" x2="87.63" y2="54.61" width="0.8128" layer="16"/>
-<wire x1="87.63" y1="51.435" x2="87.63" y2="54.61" width="0.8128" layer="16"/>
-<wire x1="87.63" y1="54.61" x2="81.28" y2="54.61" width="0.8128" layer="16"/>
+<wire x1="90.17" y1="54.61" x2="84.455" y2="54.61" width="0.8128" layer="16"/>
+<wire x1="84.455" y1="50.8" x2="84.455" y2="54.61" width="0.8128" layer="16"/>
+<wire x1="84.455" y1="54.61" x2="81.28" y2="54.61" width="0.8128" layer="16"/>
 </signal>
 <signal name="N$6">
 <contactref element="T2" pad="3"/>
 <contactref element="R5" pad="1"/>
-<wire x1="88.9" y1="46.99" x2="86.36" y2="46.99" width="0.8128" layer="16"/>
-<wire x1="86.36" y1="46.99" x2="86.36" y2="49.53" width="0.8128" layer="16"/>
+<wire x1="88.9" y1="50.8" x2="88.9" y2="49.53" width="0.8128" layer="16"/>
+<wire x1="88.9" y1="49.53" x2="86.36" y2="49.53" width="0.8128" layer="16"/>
 </signal>
 <signal name="N$7">
@@
 <wire x1="88.9" y1="17.78" x2="106.68" y2="17.78" width="0.8128" layer="16"/>
 <wire x1="85.725" y1="43.18" x2="85.725" y2="25.4" width="0.8128" layer="16"/>
-<wire x1="99.06" y1="50.8" x2="99.06" y2="46.99" width="0.8128" layer="16"/>
-<wire x1="99.06" y1="50.8" x2="99.06" y2="43.18" width="0.8128" layer="16"/>
+<wire x1="99.06" y1="48.26" x2="99.06" y2="43.18" width="0.8128" layer="16"/>
 <wire x1="99.06" y1="43.18" x2="99.06" y2="36.83" width="0.8128" layer="16"/>
 <wire x1="99.06" y1="36.83" x2="106.68" y2="36.83" width="0.8128" layer="16"/>
 <wire x1="106.68" y1="36.83" x2="106.68" y2="27.94" width="0.8128" layer="16"/>
 <wire x1="85.725" y1="43.18" x2="99.06" y2="43.18" width="0.8128" layer="16"/>
+<wire x1="99.06" y1="48.26" x2="99.06" y2="50.8" width="0" layer="19" extent="1-1"/>
 </signal>
 <signal name="VCC">
@@
 <contactref element="Q1" pad="3"/>
 <contactref element="X3" pad="1"/>
-<wire x1="109.22" y1="50.8" x2="109.22" y2="45.72" width="1.6764" layer="16"/>
+<wire x1="109.22" y1="48.26" x2="109.22" y2="45.72" width="1.6764" layer="16"/>
 <wire x1="109.22" y1="45.72" x2="109.22" y2="25.4" width="1.6764" layer="16"/>
 <wire x1="109.22" y1="25.4" x2="107.95" y2="24.13" width="1.6764" layer="16"/>
-<wire x1="105.41" y1="50.8" x2="105.37" y2="73.66" width="1.6764" layer="16"/>
+<wire x1="105.41" y1="48.26" x2="105.37" y2="73.66" width="1.6764" layer="16"/>
 <wire x1="101.6" y1="27.94" x2="101.6" y2="24.13" width="1.6764" layer="16"/>
 <wire x1="101.6" y1="24.13" x2="104.14" y2="24.13" width="1.6764" layer="16"/>
@@
 <wire x1="104.14" y1="24.13" x2="107.95" y2="24.13" width="1.6764" layer="16"/>
 <wire x1="104.14" y1="20.32" x2="104.14" y2="24.13" width="1.6764" layer="16"/>
-<wire x1="109.22" y1="50.8" x2="105.41" y2="50.8" width="1.6764" layer="16"/>
+<wire x1="109.22" y1="48.26" x2="105.41" y2="48.26" width="1.6764" layer="16"/>
 <contactref element="JP5" pad="1"/>
 <wire x1="55.88" y1="-13.97" x2="48.895" y2="-8.255" width="0.6604" layer="16"/>
@@
 <wire x1="-30.48" y1="52.705" x2="-30.48" y2="59.69" width="0.8128" layer="16"/>
 <wire x1="-30.48" y1="59.69" x2="-30.48" y2="69.215" width="0.8128" layer="16"/>
-<wire x1="-30.48" y1="69.215" x2="37.465" y2="69.215" width="0.8128" layer="16"/>
-<wire x1="37.465" y1="69.215" x2="37.465" y2="62.23" width="0.8128" layer="16"/>
-<wire x1="37.465" y1="62.23" x2="38.1" y2="62.23" width="0.8128" layer="16"/>
-<wire x1="38.1" y1="62.23" x2="38.1" y2="59.69" width="0.8128" layer="16"/>
+<wire x1="-30.48" y1="69.215" x2="38.1" y2="69.215" width="0.8128" layer="16"/>
+<wire x1="38.1" y1="69.215" x2="38.1" y2="59.69" width="0.8128" layer="16"/>
 </signal>
 <signal name="PWM_DISCHARGE1">
@@
 <wire x1="66.04" y1="54.61" x2="66.04" y2="66.04" width="0.8128" layer="16"/>
 <wire x1="66.04" y1="66.04" x2="55.88" y2="66.04" width="0.8128" layer="16"/>
-<wire x1="55.88" y1="66.04" x2="52.07" y2="66.04" width="1.27" layer="16"/>
-<wire x1="52.07" y1="66.04" x2="52.07" y2="59.69" width="1.27" layer="16"/>
-<wire x1="52.07" y1="59.69" x2="55.88" y2="59.69" width="1.27" layer="16"/>
+<wire x1="55.88" y1="66.04" x2="52.07" y2="66.04" width="0.8128" layer="16"/>
+<wire x1="52.07" y1="66.04" x2="52.07" y2="59.69" width="0.8128" layer="16"/>
+<wire x1="52.07" y1="59.69" x2="55.88" y2="59.69" width="0.8128" layer="16"/>
 <wire x1="55.88" y1="59.69" x2="55.88" y2="50.8" width="1.27" layer="16"/>
 </signal>
@@
 <contactref element="U$1" pad="D4"/>
 <contactref element="U$4" pad="2"/>
-<wire x1="45.72" y1="59.69" x2="48.26" y2="55.88" width="0.8128" layer="16"/>
-<wire x1="48.26" y1="55.88" x2="53.34" y2="55.88" width="0.8128" layer="16"/>
+<wire x1="45.72" y1="59.69" x2="46.355" y2="55.88" width="0.8128" layer="16"/>
+<wire x1="46.355" y1="55.88" x2="53.34" y2="55.88" width="0.8128" layer="16"/>
 <wire x1="53.34" y1="55.88" x2="53.34" y2="50.8" width="1.27" layer="16"/>
 <contactref element="S1" pad="3"/>
@@
 <wire x1="-38.8112" y1="40.64" x2="-38.735" y2="40.5638" width="0.8128" layer="16"/>
 <wire x1="-38.1" y1="59.69" x2="-38.1" y2="73.025" width="0.8128" layer="16"/>
-<wire x1="-38.1" y1="73.025" x2="45.085" y2="73.025" width="0.8128" layer="16"/>
-<wire x1="45.085" y1="73.025" x2="45.085" y2="59.69" width="0.8128" layer="16"/>
-<wire x1="45.085" y1="59.69" x2="45.72" y2="59.69" width="0.8128" layer="16"/>
+<wire x1="-38.1" y1="73.025" x2="45.72" y2="73.025" width="0.8128" layer="16"/>
+<wire x1="45.72" y1="73.025" x2="45.72" y2="59.69" width="0.8128" layer="16"/>
 </signal>
 <signal name="N$30">
@@
 <wire x1="62.23" y1="40.64" x2="62.23" y2="35.56" width="0.6604" layer="16"/>
 <wire x1="62.23" y1="35.56" x2="64.77" y2="35.56" width="0.6604" layer="16"/>
-<wire x1="72.39" y1="73.66" x2="72.39" y2="66.04" width="0.6604" layer="16"/>
+<wire x1="72.39" y1="73.66" x2="72.39" y2="66.04" width="0.8128" layer="16"/>
 <wire x1="72.39" y1="60.96" x2="72.39" y2="48.26" width="0.6604" layer="16"/>
 <wire x1="72.39" y1="73.66" x2="72.51" y2="73.66" width="0.6604" layer="16"/>

Commit message: renumbered
Parts:
- removed C8: 100n, rcl:C025_050-025X075
- removed R39: 1R666, rcl:0414/15
- added C7: 10µ, rcl:E5-5
- added R10: 2k2, rcl:0207/15
- C1, C6: value 10µ -> 100n; device rcl:E5-5 -> rcl:C025_050-025X075
- C4: value 100n -> 3µ3; device rcl:C025_050-025X075 -> rcl:E5-5
- C5: value 3µ3 -> 10µ
- IC1: value LM324N -> TL431; device linear:DIL14 -> AWJLEagleLib:TO92
- IC2: value TL431 -> LM324N; device AWJLEagleLib:TO92 -> linear:DIL14
- JP1, JP2, JP6, JP8: device bigger:JP1 -> bigger:JP2
- JP16, JP17, JP18, JP9: device bigger:JP2 -> bigger:JP1
- LED2: value (none) -> CHRG2
- LED3: value CHRG2 -> (none)
- Q1: value BD648 -> BUZ11; device transistor-pnp:TO220 -> transistor-fet:TO220
- Q2: value BUZ11 -> BD648; device transistor-fet:TO220 -> transistor-pnp:TO220
- R1: value 470 -> 4k7; device rcl:0207/12 -> rcl:0204/7
- R11: value 100k -> 1k; device rcl:0207/10 -> rcl:0204/7
- R12: value 1k -> 1R666; device rcl:0207/12 -> rcl:0414/15
- R14: value 10k -> 0
- R15: value 100k -> 1k
- R16: value 33k -> 1k
- R17: value 1k -> 12k; device rcl:0207/15 -> rcl:0207/10
- R18: value 12k -> 100k
- R19: value 1k -> 33k; device rcl:0204/7 -> rcl:0207/10
- R2: value 100k -> 4k7; device rcl:0204/7 -> rcl:0207/10
- R20: value 470 -> 1k; device rcl:0207/10 -> rcl:0207/15
- R21: value 200 -> 1k; device rcl:0204/7 -> rcl:0207/12
- R22: value 4k7 -> 200; device rcl:0207/10 -> rcl:0207/12
- R23: value 470 -> 1M
- R24: value 0 -> 100k; device rcl:0207/10 -> rcl:0204/7
- R25: value 4k7 -> 1k; device rcl:0204/7 -> rcl:0207/10
- R26: value 470 -> 100k
- R27: value 470 -> 10k; device rcl:0204/7 -> rcl:0207/10
- R28: value 0 -> 10k; device rcl:0204/7 -> rcl:0207/10
- R29: value 0 -> 1k; device rcl:0204/7 -> rcl:0207/12
- R3: device rcl:0207/10 -> rcl:0207/12
- R30: value 0 -> 100k; device rcl:0204/7 -> rcl:0207/10
- R31: value 0 -> 1R666; device rcl:0204/7 -> rcl:0414/15
- R33: device rcl:0204V -> rcl:0204/7
- R34: device rcl:0204/7 -> rcl:0204V
- R35: value 100k -> 0
- R36: value 1M -> 0; device rcl:0207/10 -> rcl:0204/7
- R37: value 200 -> 0; device rcl:0207/12 -> rcl:0204/7
- R38: value 1k -> 0; device rcl:0207/10 -> rcl:0204/7
- R4: value 2k2 -> 200; device rcl:0207/15 -> rcl:0204/7
- R5, R6: value 1k -> 470
- R7: value 1R666 -> 470; device rcl:0414/15 -> rcl:0207/10
- R8: value 1k -> 470; device rcl:0207/12 -> rcl:0204/7
- R9: value 10k -> 470; device rcl:0207/10 -> rcl:0204/7
- S4: value Discharge -> A
- S5: value A -> B
- S6: value B -> Discharge
- U$1: value ARDUINOR3BPLACE-LONG -> DS1820TO92; device arduino-long:ARDUINOR3-BPLACE-LONG -> Ava:DS1820
- U$2: value DS1820TO92 -> ARDUINOR3BPLACE-LONG; device Ava:DS1820 -> arduino-long:ARDUINOR3-BPLACE-LONG
- X2: value Battery -> VCC; device con-wago-500:W237-6 -> con-wago-500:W237-102
- X3: value VCC -> Battery; device con-wago-500:W237-102 -> con-wago-500:W237-6
- moved R6 139.2 mm to (-21.6, -11.4), turned to 180 degrees
- moved R5 130.1 mm to (-21.6, -8.89)
- moved R23 113.8 mm to (71.1, 52.1), turned to 0 degrees
- moved JP16 91.1 mm to (78.7, 61.0), turned to 270 degrees
- moved R8 89.2 mm to (-6.99, 50.8), turned to 0 degrees
- moved JP17 88.9 mm to (71.1, 61.0), turned to 90 degrees
- moved R20 83.7 mm to (55.9, 20.3), turned to 270 degrees
- moved JP2 79.6 mm to (8.89, -7.62), turned to 0 degrees
- moved R31 79.5 mm to (77.5, 66.0)
- moved JP23 76.8 mm to (11.4, 12.7), turned to 180 degrees
- moved R26 75.6 mm to (59.7, 15.2), turned to 90 degrees
- moved JP24 75.5 mm to (11.4, 26.7), turned to 0 degrees
- moved R7 75.0 mm to (-21.6, -14.0)
- moved R9 73.9 mm to (-6.99, 48.3), turned to 0 degrees
- moved U$3 73.7 mm to (40.6, 59.7), turned to 180 degrees
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- renumbered T2 to T1
Connections:
- net +5V: now also JP20.1, JP3.1, JP3.2, JP6.3, JP8.3, R1.2, R4.2, U$1.VDD, U$2.5V; no longer JP16.1, JP16.2, JP16.3, JP5.3, JP9.1, R21.2, R25.2, U$1.5V, U$2.VDD
- net 3V: now also U$2.3V; no longer U$1.3V
- net GND: now also C1.2, C4.-, C7.-, IC1.2, IC2.11, JP17.2, JP2.1, JP2.2, JP2.3, JP20.3, JP4.2, JP6.1, R12.2, R17.1, R19.1, R23.1, R25.1, R26.1, R30.1, R31.2, R32.2, R33.2, R37.2, U$2.GND1, U$2.GND2, X2.2, X3.6; no longer C1.-, C4.2, C6.-, IC1.11, IC2.2, JP18.1, JP18.2, JP18.3, JP22.2, JP23.2, JP3.1, JP9.3, R11.1, R16.1, R18.1, R28.2, R29.2, R34.2, R35.1, R36.1, R38.1, R39.2, R7.2, U$1.GND1, U$1.GND2, X2.6, X3.2
- net I1_SENSE+: now also JP16.2, R31.1, X3.3; no longer JP24.2, R39.1, X2.3
- net I1_SENSE-: now also JP17.1, R28.1, X3.5; no longer JP23.1, R9.1, X2.5
- net I_BATT1: now also C4.+, R21.1, U$2.A1; no longer C2.+, R12.1, U$1.A1
- net I_BATT2: now also JP5.2, U$2.A4; no longer JP20.2, U$1.A4
- net I_DISC1: now also R20.2, U$2.A2; no longer R17.2, U$1.A2
- net I_DISC2: now also JP5.3, U$2.A5; no longer JP20.3, U$1.A5
- net N$1: now also R3.2, U$2.D13; no longer R1.2, U$1.D13
- net N$10: now also C6.1, JP13.1; no longer C8.1, JP1.1
- net N$11: now also IC2.1, JP12.2, R24.2; no longer IC1.1, JP7.2, R2.2
- net N$12: now also JP6.2, R1.1, U$1.DQ, U$2.D2; no longer JP3.2, R25.1, U$1.D2, U$2.DQ
- net N$13: now also JP13.2, JP15.2, Q1.2, X3.2; no longer JP1.2, JP2.2, Q2.2, X2.2
- net N$14: now also IC2.2, R24.1, R28.2; no longer IC1.2, R2.1, R9.2
- net N$15: now also IC2.3, R26.2, R27.1; no longer IC1.3, R14.1, R35.2
- net N$16: now also IC2.6, R17.2, R18.1, R19.2; no longer IC1.6, R15.1, R16.2, R18.2
- net N$17: now also IC2.7, JP11.1, R18.2; no longer IC1.7, JP15.1, R15.2
- net N$18: now also Q1.1, R11.2; no longer Q2.1, R19.2
- net N$19: now also R5.2, U$2.D5; no longer R3.2, U$1.D5
- net N$2: now also R3.1; no longer R1.1
- net N$20: now also LED3.A, R6.2; no longer LED2.A, R20.2
- net N$21: now also R7.2; no longer R23.2
- net N$22: now also JP14.1, R27.2; no longer JP6.1, R14.2
- net N$23: now also S6.3, U$2.D12; no longer S4.3, U$1.D12
- net N$24: now also LED2.A, R5.1; no longer LED3.A, R3.1
- net N$25: now also JP10.1, Q1.3, R12.1; no longer JP8.1, Q2.3, R7.1
- net N$26: now also U$2.D4; no longer U$1.D4
- net N$27: now also IC1.1, IC1.3, R2.2, R4.1; no longer IC2.1, IC2.3, R21.1, R22.2
- net N$28: now also R2.1, U$2.AREF; no longer R22.1, U$1.AREF
- net N$29: now also C2.+, IC2.5, R14.1; no longer C5.+, IC1.5, R24.1
- net N$3: now also C7.+, JP18.1, R29.2, R30.2; no longer C1.+, JP4.1, R13.2, R8.2
- net N$30: now also U$2.D7; no longer U$1.D7
- net N$31: now also U$2.D8; no longer U$1.D8
- net N$32: now also JP12.1, R21.2; no longer JP7.1, R12.2
- net N$33: now also JP10.2, R14.2; no longer JP8.2, R24.2
- net N$34: now also IC2.8, JP21.1, R34.1; no longer IC1.8, JP11.1, R33.1
- net N$35: now also JP11.2, R20.1; no longer JP15.2, R17.1
- net N$36: now also IC2.13, R36.1, R37.1; no longer IC1.13, R29.1, R31.1
- net N$37: now also S4.3, U$2.D6; no longer S5.3, U$1.D6
- net N$38: now also S5.3, U$2.SDA; no longer S6.3, U$1.SDA
- net N$39: now also R8.2; no longer R26.2
- net N$4: now also C1.1, IC2.4, JP8.2; no longer C4.1, IC1.4, JP5.2
- net N$40: now also R9.2; no longer R27.2
- net N$41: now also R9.1, U$2.SCL; no longer R27.1, U$1.SCL
- net N$42: now also JP7.2, R8.1, U$2.D1; no longer JP21.2, R26.1, U$1.D1
- net N$43: now also IC2.10, JP19.2; no longer IC1.10, JP10.2
- net N$44: now also JP19.1, R32.1; no longer JP10.1, R28.1
- net N$45: now also IC2.12, R35.1, R38.2; no longer IC1.12, R30.1, R32.2
- net N$46: now also JP22.1, JP22.2, R35.2; no longer JP12.1, JP12.2, R30.2
- net N$47: now also JP23.1, JP23.2, R36.2; no longer JP13.1, JP13.2, R31.2
- net N$48: now also IC2.14, JP24.1, JP24.2, R38.1; no longer IC1.14, JP14.1, JP14.2, R32.1
- net N$49: now also IC2.9, R33.1, R34.2; no longer IC1.9, R33.2, R34.1
- net N$5: now also R10.2, R13.2; no longer R11.2, R4.2
- net N$50: now also C6.2, R25.2; no longer C8.2, R38.2
- net N$51: now also R22.2, R23.2; no longer R36.2, R37.2
- net N$52: now also JP7.1, U$2.D0; no longer JP21.1, U$1.D0
- net N$53: now also JP4.1, U$2.RESET; no longer JP22.1, U$1.RESET
- net N$54: now also JP14.2, JP16.1, X3.4; no longer JP24.1, JP6.2, X2.4
- net N$6: now also R15.1; no longer R5.1
- net N$7: now also Q2.1, R15.2, R16.1; no longer Q1.1, R5.2, R6.1
- net N$8: now also JP15.1, R29.1, X3.1; no longer JP2.1, R8.1, X2.1
- net N$9: now also Q2.2; no longer Q1.2
- net PWM_CHARGE1: now also R10.1, U$2.D3; no longer R4.1, U$1.D3
- net PWM_CHARGE2: now also R22.1, U$2.D11; no longer R37.1, U$1.D11
- net PWM_DISCHARGE1: now also R11.1, R6.1, U$2.D10; no longer R19.1, R20.1, U$1.D10
- net PWM_DISCHARGE2: now also R7.1, U$2.D9; no longer R23.1, U$1.D9
- net U_BATT1: now also JP18.2, U$2.A0; no longer JP4.2, U$1.A0
- net U_BATT2: now also JP5.1, U$2.A3; no longer JP20.1, U$1.A3
- net VCC: now also C5.+, JP20.2, JP8.1, JP9.1, Q2.3, R16.2, X2.1; no longer C6.+, JP19.1, JP5.1, JP9.2, Q1.3, R6.2, X3.1
- net VIN: now also JP1.1, JP1.2, JP1.3, JP9.2, U$2.VIN; no longer JP17.1, JP17.2, JP17.3, JP19.2, U$1.VIN

Commit message: v1
Parts:
- moved JP4 2.54 mm to (33.0, -8.89)
- moved JP20 2.54 mm to (29.2, -7.62)
- moved Q1 1.27 mm to (80.0, -7.62)
- moved R12 1.27 mm to (53.3, -10.2)
Routing:
- net GND: track 195.0 -> 164.6 mm
- net VIN: track 70.4 -> 57.7 mm
- net N$25: track 69.6 -> 60.7 mm
- net VCC: track 232.8 -> 228.2 mm
- net +5V: track 121.1 -> 124.4 mm
- net N$7: track 88.3 -> 90.9 mm
- net N$53: track 7.62 -> 10.2 mm
- net PWM_DISCHARGE1: track 170.7 -> 172.4 mm
- net N$1: track 101.5 -> 102.9 mm
- net N$18: track 84.9 -> 83.6 mm
- net N$13: track 126.2 -> 125.0 mm

Commit message: before production
Parts:
- added R39: *, rcl:0204/7
- R21: device rcl:0207/12 -> rcl:0204/7
- moved R21 2.54 mm to (49.5, 11.4)
- moved C2 0.32 mm to (40.6, 17.5)
- moved R14 0.32 mm to (40.6, 21.3)
Connections:
- net GND: now also R39.1
- net N$32: now also R39.2
Routing:
- net N$32: track 3.81 -> 13.8 mm
- net N$31: track 170.3 -> 169.2 mm
- net N$29: track 15.0 -> 15.7 mm
Other:
- board text added: "ChargerShieldExpA"
- board text added: "v1"
