File: Production/V1/ChargerShieldExpA.brd (EAGLE design)
At the start: 160 x 99.1 mm, 102 parts, among them IC1 TL431, IC2 LM324N, Q1 BUZ11, Q2 BD648, Q3 BUZ171, Q4 IRFZ48Z, T1 BC548, X1 +Vin, X2 VCC, X3 Battery

Commit message: V1 Production review
Parts:
- removed JP25: (no value), bigger:JP1
- R35: device rcl:0207/10 -> rcl:0204/7
- moved R16 3.81 mm to (104.1, 48.3)
- moved R5 2.54 mm to (-21.6, -8.89)
- moved C5 1.91 mm to (104.1, 45.7)
- moved R35 1.27 mm to (8.26, 17.8)
- moved R37 1.27 mm to (15.2, 19.1)
- moved R6 1.27 mm to (-21.6, -11.4)
- moved R15 1.27 mm to (94.0, 50.8)
- moved L1 0.64 mm to (81.3, 27.9)
- moved R11 0.32 mm to (36.2, 40.0)
- moved R39 0.16 mm to (39.4, 12.7)
- moved R1 0.16 mm to (39.4, 38.7)
Connections:
- removed net N$64: JP25.1, R2.1
- net N$28: now also R2.1; no longer JP25.2
Routing:
- net N$48: track 23.7 -> 37.4 mm
- net N$28: track 15.3 -> 4.04 mm
- net N$64: track 6.61 -> 0.00 mm
- net N$38: track 158.7 -> 164.2 mm
- net N$7: track 95.9 -> 90.9 mm
- net GND: track 169.3 -> 164.6 mm
- net PWM_DISCHARGE2: track 192.6 -> 187.9 mm
- net N$24: track 12.7 -> 15.2 mm
- net N$19: track 181.4 -> 183.9 mm
- net N$36: track 7.92 -> 6.35 mm
- net N$31: track 167.7 -> 169.2 mm
- net N$34: track 10.1 -> 8.56 mm
- net N$39: track 76.4 -> 75.0 mm
- net N$26: track 146.7 -> 148.0 mm
- net N$23: track 144.9 -> 146.2 mm
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Other:
- outline, holes or cut-outs redrawn
- board text added: "ChargerShieldExpA"
- board text removed: "ChgShieldExpA"
